File: hardware/button_board/northreach_1_button_board.kicad_pcb (KiCad board)
At the start: 2 copper layers, 0 parts

Commit message: pcb: button board: layout
Parts:
- added C6: 0.1uF, Capacitor_SMD:C_0805_2012Metric, F.Cu at (67.2, 131.7)
- added D1: WS2812B, LED_SMD:LED_WS2812B_PLCC4_5.0x5.0mm_P3.2mm, F.Cu at (73.0, 132.3)
- added H1: MountingHole_Pad, MountingHole:MountingHole_2.2mm_M2_Pad, F.Cu at (60.5, 56.5)
- added H2: MountingHole_Pad, MountingHole:MountingHole_2.2mm_M2_Pad, F.Cu at (85.5, 56.5)
- added H3: MountingHole_Pad, MountingHole:MountingHole_2.2mm_M2_Pad, F.Cu at (60.5, 136.5)
- added H4: MountingHole_Pad, MountingHole:MountingHole_2.2mm_M2_Pad, F.Cu at (85.5, 136.5)
- added J1: Conn_01x20, Connector_FFC-FPC:Hirose_FH12-20S-0.5SH_1x20-1MP_P0.50mm_Horizontal, F.Cu at (73.0, 139.0)
- added SW10: Fn_1, Button_Switch_THT:SW_PUSH_6mm_H5mm, F.Cu at (61.8, 110.2)
- added SW11: Fn_2, Button_Switch_THT:SW_PUSH_6mm_H5mm, F.Cu at (77.8, 110.2)
- added SW12: Fn_3, Button_Switch_THT:SW_PUSH_6mm_H5mm, F.Cu at (61.8, 122.2)
- added SW13: Fn_4, Button_Switch_THT:SW_PUSH_6mm_H5mm, F.Cu at (77.8, 122.2)
- added SW3: Left, Button_Switch_THT:SW_PUSH_6mm_H5mm, F.Cu at (57.6, 68.2)
- added SW4: Right, Button_Switch_THT:SW_PUSH_6mm_H5mm, F.Cu at (81.9, 68.2)
- added SW5: Up, Button_Switch_THT:SW_PUSH_6mm_H5mm, F.Cu at (69.8, 56.2)
- added SW6: Vol_Up, Button_Switch_THT:SW_PUSH_6mm_H5mm, F.Cu at (61.8, 94.7)
- added SW7: Down, Button_Switch_THT:SW_PUSH_6mm_H5mm, F.Cu at (69.8, 80.3)
- added SW8: Vol_Down, Button_Switch_THT:SW_PUSH_6mm_H5mm, F.Cu at (77.8, 94.7)
- added SW9: Return, Button_Switch_THT:SW_PUSH_6mm_H5mm, F.Cu at (69.8, 68.2)
Routing:
- added copper zone on B.Cu, net GND
Other:
- board outline added: 41 x 96 mm

Commit message: pcb: button board: routing
Parts:
- moved D1 81.4 mm to (136.4, 81.2)
- moved C6 81.2 mm to (130.3, 80.6)
- moved H1 74.9 mm to (135.4, 55.1)
- moved H2 74.9 mm to (160.4, 55.1)
- moved H3 74.9 mm to (135.4, 135.1)
- moved H4 74.9 mm to (160.4, 135.1)
- moved J1 74.9 mm to (147.9, 137.6)
- moved SW10 74.9 mm to (136.7, 108.8)
- moved SW11 74.9 mm to (152.7, 108.8)
- moved SW12 74.9 mm to (136.7, 120.8)
- moved SW13 74.9 mm to (152.7, 120.8)
- moved SW5 74.9 mm to (144.7, 54.9)
- moved SW6 74.9 mm to (136.7, 93.2)
- moved SW7 74.9 mm to (144.7, 79.0)
- moved SW8 74.9 mm to (152.7, 93.2)
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Routing:
- net BUTTON_LEFT: track 0.00 -> 141.8 mm
- net BUTTON_RETURN: track 0.00 -> 118.0 mm
- net BUTTON_UP: track 0.00 -> 109.0 mm
- net BUTTON_VOL_DOWN: track 0.00 -> 87.8 mm
- net BUTTON_DOWN: track 0.00 -> 87.4 mm
- net BUTTON_RIGHT: track 0.00 -> 87.2 mm
- net STATUS_LED_DATA: track 0.00 -> 80.0 mm
- net VBUS: track 0.00 -> 73.3 mm
- net BUTTON_FN_1: track 0.00 -> 72.6 mm
- net BUTTON_VOL_UP: track 0.00 -> 65.9 mm
- net BUTTON_FN_4: track 0.00 -> 58.2 mm
- net BUTTON_FN_2: track 0.00 -> 48.5 mm
- net BUTTON_FN_3: track 0.00 -> 23.9 mm
- net GND: track 0.00 -> 7.59 mm, vias 0 -> 3
