File: hardware/button_board/northreach_1_button_board.kicad_pcb (KiCad board)
At the start: 2 copper layers, 41 x 96 mm, 16 parts, among them J1 Conn_01x20, SW10 Fn_1, SW11 Fn_2, SW12 Fn_3, SW13 Fn_4, SW3 Left, SW4 Right, SW5 Up, SW6 Vol_Up, SW7 Down, SW8 Vol_Down, SW9 Return

Commit message: pcb: button board: silkscreen
Other:
- board text added: "NorthReach 1 - Button Board v1 - Designed on Jan. 8th 2026 in Athens, Greece Stratos Thivaios (C) 2026"
- board text added: "NorthReach 1 - v1 Stratos Thivaios (C) 2026"
- board text removed: "NorthReach 1 - Button Board v1 - Designed on Jan. 8th 2025 in Athens, Greece Stratos Thivaios (C) 2025"
- board text removed: "NorthReach 1 - v1 Stratos Thivaios (C) 2025"
Changed lines of the file:
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@@
 		(layer "Edge.Cuts")
 	)
-	(gr_text "NorthReach 1 - v1\nStratos Thivaios (C) 2025"
+	(gr_text "NorthReach 1 - v1\nStratos Thivaios (C) 2026"
 		(at 148 50 0)
 		(layer "F.SilkS")
@@
 		)
 	)
-	(gr_text "NorthReach 1 - Button Board\nv1 - Designed on Jan. 8th 2025\nin Athens, Greece\nStratos Thivaios (C) 2025"
+	(gr_text "NorthReach 1 - Button Board\nv1 - Designed on Jan. 8th 2026\nin Athens, Greece\nStratos Thivaios (C) 2026"
 		(at 148 134 0)
 		(layer "B.SilkS")

Commit message: schematic_and_pcb: button board: SW numbering
Parts:
- renumbered SW3 to SW1, SW6 to SW10, SW8 to SW11, SW4 to SW2, SW5 to SW3, SW7 to SW4, SW9 to SW5, SW10 to SW6, SW11 to SW7, SW12 to SW8, SW13 to SW9
